Commit message: Versión 2.0

File: src/enjambre_drones/urdf/dron_base.xacro (robot description, xacro)
@@ -1,81 +1,196 @@
 <?xml version="1.0"?>
 <!--
-  ========================================================================
-  ROBOT: Drone X (Quadcopter) - Base para enjambre de drones
-  Autor: TFG Control de Enjambres - FP ROS2
-  Descripción:
-    Modelo XACRO de un cuadricóptero en configuración "X" con:
-    - Cuerpo central, brazos, motores, hélices, patas y LED superior.
-    - Materiales diferenciados por zonas (frontal/trasero).
-    - Inercias simples para simulación ligera.
-    - Diseñado para ser usado en Gazebo y RViz.
-    - El LED central puede cambiar de color mediante un tópico ROS2.
-  ========================================================================
+  dron_base.xacro
+  ============================================================================-
+  Modelo Xacro/URDF de un dron cuadricóptero para ROS 2 y RViz.
+  Objetivo del fichero:
+  - Dibujar el cuerpo central del dron.
+  - Dibujar los cuatro brazos diagonales.
+  - Dibujar los cuatro motores.
+  - Dibujar las hélices de cada motor.
+  - Dibujar un LED superior de estado.
+  - Dibujar cuatro patas reales de aterrizaje, una en cada esquina del cuerpo.
+  - Permitir instanciar varios drones iguales usando un prefijo distinto.
+  Por qué usamos prefix:
+  ============================================================================-
+  Si lanzamos seis drones en RViz, todos tendrían nombres de enlaces repetidos:
+  base_link, status_led_link, front_left_motor_link, etc.
+  Eso genera conflictos en TF. Por eso todos los nombres de links y joints usan:
+      ${prefix}
+  De esta forma, al lanzar el dron con prefix:=drone1_, se generan nombres como:
+      drone1_base_link
+      drone1_status_led_link
+      drone1_front_left_motor_link
+  y con prefix:=drone2_:
+      drone2_base_link
+      drone2_status_led_link
+      drone2_front_left_motor_link
+  Así cada dron tiene su propio árbol TF.
+  Nota sobre el LED:
+  ============================================================================-
+  Este fichero dibuja un LED físico fijo sobre el cuerpo del dron.
+  Para cambiar dinámicamente el color desde ROS 2, en la versión RViz es más
+  sencillo usar MarkerArray desde swarm_visualizer.py. El LED del Xacro queda
+  como referencia visual del modelo.
 -->
 <robot xmlns:xacro="http://www.ros.org/wiki/xacro" name="drone_x_led">
-  <!-- ==================================================================== -->
-  <!-- 1. PROPIEDADES GEOMÉTRICAS Y DE POSICIONAMIENTO                      -->
-  <!-- ==================================================================== -->
-  <!-- Constantes auxiliares -->
-  <xacro:property name="diag" value="0.70710678"/>  <!-- sqrt(2)/2, útil para diagonales -->
-  <!-- Dimensiones del cuerpo principal -->
-  <xacro:property name="body_l" value="0.16"/>
-  <xacro:property name="body_w" value="0.16"/>
-  <xacro:property name="body_h" value="0.045"/>
-  <!-- Dimensiones de los brazos -->
-  <xacro:property name="arm_l" value="0.20"/>
-  <xacro:property name="arm_w" value="0.014"/>
-  <xacro:property name="arm_h" value="0.014"/>
-  <xacro:property name="arm_inside" value="0.025"/>  <!-- Distancia desde el cuerpo hasta inicio del brazo -->
-  <!-- Dimensiones del motor -->
-  <xacro:property name="motor_r" value="0.022"/>
-  <xacro:property name="motor_h" value="0.028"/>
-  <!-- Dimensiones de la hélice -->
-  <xacro:property name="prop_l" value="0.15"/>
-  <xacro:property name="prop_w" value="0.016"/>
-  <xacro:property name="prop_h" value="0.005"/>
-  <xacro:property name="prop_hub_r" value="0.010"/>
-  <xacro:property name="prop_hub_h" value="0.008"/>
-  <!-- Patas -->
-  <xacro:property name="leg_r" value="0.006"/>
-  <xacro:property name="leg_h" value="0.10"/>
-  <!-- LED central -->
+  <!-- ======================================================================= -->
+  <!-- 1. ARGUMENTOS DEL MODELO                                                -->
+  <!-- ======================================================================= -->
+  <!--
+    prefix permite crear varios drones iguales sin que se repitan los nombres
+    de los links y joints.
+    Ejemplos:
+      prefix:=drone1_
+      prefix:=drone2_
+      prefix:=drone3_
+  -->
+  <xacro:arg name="prefix" default=""/>
+  <xacro:property name="prefix" value="$(arg prefix)"/>
+  <!-- ======================================================================= -->
+  <!-- 2. CONSTANTES GEOMÉTRICAS GENERALES                                     -->
+  <!-- ======================================================================= -->
+  <!--
+    Valor aproximado de cos(45º) y sin(45º).
+    Se usa para colocar los brazos en diagonal, formando una X.
+  -->
+  <xacro:property name="diag" value="0.70710678"/>
+  <!-- ======================================================================= -->
+  <!-- 3. DIMENSIONES DEL CUERPO CENTRAL                                       -->
+  <!-- ======================================================================= -->
+  <!--
+    El cuerpo central se representa como una caja.
+    Ejes usados en RViz/URDF:
+      X: delante / atrás
+      Y: izquierda / derecha
+      Z: arriba / abajo
+  -->
+  <xacro:property name="body_l" value="0.16"/>   <!-- Longitud del cuerpo en X -->
+  <xacro:property name="body_w" value="0.16"/>   <!-- Anchura del cuerpo en Y  -->
+  <xacro:property name="body_h" value="0.045"/>  <!-- Altura del cuerpo en Z   -->
+  <!-- ======================================================================= -->
+  <!-- 4. DIMENSIONES DE LOS BRAZOS                                            -->
+  <!-- ======================================================================= -->
+  <!--
+    Cada brazo se representa como una barra rectangular.
+    Los brazos salen desde el cuerpo hacia las cuatro esquinas.
+  -->
+  <xacro:property name="arm_l" value="0.20"/>       <!-- Longitud de cada brazo -->
+  <xacro:property name="arm_w" value="0.014"/>      <!-- Grosor lateral del brazo -->
+  <xacro:property name="arm_h" value="0.014"/>      <!-- Altura del brazo -->
+  <xacro:property name="arm_inside" value="0.025"/> <!-- Parte del brazo que entra visualmente en el cuerpo -->
+  <!--
+    arm_center_offset calcula cuánto hay que desplazar el centro de cada brazo
+    para que quede correctamente unido al cuerpo y orientado en diagonal.
+  -->
+  <xacro:property name="arm_center_offset" value="${(arm_l/2.0 - arm_inside) * diag}"/>
+  <!--
+    Altura a la que se colocan los brazos.
+    Se sitúan encima del cuerpo central, no atravesando su centro.
+  -->
+  <xacro:property name="arm_z" value="${body_h/2.0 + arm_h/2.0}"/>
+  <!-- ======================================================================= -->
+  <!-- 5. DIMENSIONES DE LOS MOTORES                                           -->
+  <!-- ======================================================================= -->
+  <!--
+    Cada motor se representa como un cilindro situado al final de cada brazo.
+  -->
+  <xacro:property name="motor_r" value="0.022"/>  <!-- Radio del cilindro del motor -->
+  <xacro:property name="motor_h" value="0.028"/>  <!-- Altura del cilindro del motor -->
+  <!-- ======================================================================= -->
+  <!-- 6. DIMENSIONES DE LAS HÉLICES                                           -->
+  <!-- ======================================================================= -->
+  <!--
+    Cada hélice se representa de forma sencilla:
+      - un buje central cilíndrico,
+      - dos palas rectangulares cruzadas a 90 grados.
+    No buscamos aerodinámica real, sino una representación visual clara.
+  -->
+  <xacro:property name="prop_l" value="0.15"/>      <!-- Longitud de cada pala -->
+  <xacro:property name="prop_w" value="0.016"/>     <!-- Anchura de cada pala -->
+  <xacro:property name="prop_h" value="0.005"/>     <!-- Grosor de cada pala -->
+  <xacro:property name="prop_hub_r" value="0.010"/> <!-- Radio del buje central -->
+  <xacro:property name="prop_hub_h" value="0.008"/> <!-- Altura del buje central -->
+  <!-- ======================================================================= -->
+  <!-- 7. DIMENSIONES DE LAS CUATRO PATAS DE ATERRIZAJE                        -->
+  <!-- ======================================================================= -->
+  <!--
+    En esta versión NO usamos dos cilindros largos como patines.
+    En su lugar se dibujan cuatro patas independientes:
+      - front_left_leg_link
+      - front_right_leg_link
+      - rear_left_leg_link
+      - rear_right_leg_link
+    Cada pata tiene:
+      - un cilindro vertical estrecho,
+      - una pequeña base circular inferior para simular el apoyo en el suelo.
+  -->
+  <xacro:property name="leg_r" value="0.006"/>       <!-- Radio de cada pata vertical -->
+  <xacro:property name="leg_h" value="0.090"/>       <!-- Altura de cada pata vertical -->
+  <xacro:property name="foot_r" value="0.018"/>      <!-- Radio del pequeño pie inferior -->
+  <xacro:property name="foot_h" value="0.008"/>      <!-- Altura del pequeño pie inferior -->
+  <!--
+    Posición de las patas respecto al centro del cuerpo.
+    Se colocan cerca de las cuatro esquinas inferiores del cuerpo.
+  -->
+  <xacro:property name="leg_x" value="0.055"/>       <!-- Separación de la pata respecto al centro en X -->
+  <xacro:property name="leg_y" value="0.055"/>       <!-- Separación de la pata respecto al centro en Y -->
+  <!-- ======================================================================= -->
+  <!-- 8. DIMENSIONES DEL LED DE ESTADO                                        -->
+  <!-- ======================================================================= -->
+  <!--
+    El LED se representa como una esfera pequeña sobre la parte superior del dron.
+    En RViz, el cambio dinámico de color puede representarse mejor con MarkerArray.
+  -->
   <xacro:property name="led_r" value="0.012"/>
-  <!-- Cálculos derivados -->
-  <!-- Desplazamiento del centro del brazo respecto a la esquina del cuerpo -->
-  <xacro:property name="arm_center_offset" value="${(arm_l/2.0 - arm_inside) * diag}"/>
-  <!-- Altura a la que se apoyan los brazos sobre el cuerpo -->
-  <xacro:property name="arm_z" value="${body_h/2.0 + arm_h/2.0}"/>
-  <!-- ==================================================================== -->
-  <!-- 2. MATERIALES (VISUALIZACIÓN EN RViz Y GAZEBO)                      -->
-  <!-- ==================================================================== -->
+  <!-- ======================================================================= -->
+  <!-- 9. MATERIALES Y COLORES                                                 -->
+  <!-- ======================================================================= -->
+  <!--
+    Los materiales se aplican a las geometrías visuales.
+    rgba = rojo verde azul alfa
+    El alfa 1.0 indica que el objeto es totalmente opaco.
+  -->
+  <!-- Color oscuro para el cuerpo principal. -->
   <material name="body_mat">
-    <color rgba="0.10 0.10 0.10 1.0"/>  <!-- Cuerpo negro mate -->
-  </material>
+    <color rgba="0.10 0.10 0.10 1.0"/>
+  </material>
+  <!-- Color gris para los brazos. -->
   <material name="arm_mat">
-    <color rgba="0.70 0.70 0.70 1.0"/>  <!-- Brazos gris plata -->
-  </material>
+    <color rgba="0.70 0.70 0.70 1.0"/>
+  </material>
+  <!-- Color oscuro para los motores. -->
   <material name="motor_mat">
-    <color rgba="0.12 0.12 0.12 1.0"/>  <!-- Motores negros -->
-  </material>
+    <color rgba="0.12 0.12 0.12 1.0"/>
+  </material>
+  <!-- Color rojo para las hélices delanteras. Ayuda a identificar el frontal. -->
   <material name="front_prop_mat">
-    <color rgba="0.90 0.22 0.22 1.0"/>  <!-- Hélices delanteras rojas -->
-  </material>
+    <color rgba="0.90 0.22 0.22 1.0"/>
+  </material>
+  <!-- Color azul para las hélices traseras. Ayuda a identificar la parte trasera. -->
   <material name="rear_prop_mat">
-    <color rgba="0.20 0.35 0.95 1.0"/>  <!-- Hélices traseras azules -->
-  </material>
+    <color rgba="0.20 0.35 0.95 1.0"/>
+  </material>
+  <!-- Color gris claro para las patas de aterrizaje. -->
   <material name="leg_mat">
-    <color rgba="0.80 0.80 0.80 1.0"/>  <!-- Patas gris claro -->
-  </material>
-  <!-- Material por defecto para el LED (se puede sobrescribir desde Python) -->
+    <color rgba="0.80 0.80 0.80 1.0"/>
+  </material>
+  <!-- Color ligeramente más claro para los pies inferiores de apoyo. -->
+  <material name="foot_mat">
+    <color rgba="0.90 0.90 0.90 1.0"/>
+  </material>
+  <!-- Color base del LED físico dibujado en el Xacro. -->
   <material name="led_green_mat">
-    <color rgba="0.10 1.00 0.10 1.0"/>  <!-- Verde brillante -->
-  </material>
-  <!-- ==================================================================== -->
-  <!-- 3. MACRO DE INERCIA SIMPLIFICADA                                     -->
-  <!-- ==================================================================== -->
-  <!--
-    Para simulación ligera se usa una inercia fija.
-    En un proyecto real se podría calcular con la geometría.
+    <color rgba="0.10 1.00 0.10 1.0"/>
+  </material>
+  <!-- ======================================================================= -->
+  <!-- 10. MACRO DE INERCIA SIMPLE                                             -->
+  <!-- ======================================================================= -->
+  <!--
+    Esta macro añade una inercia sencilla a cada link.
+    En RViz la inercia no es importante para visualizar el modelo, pero en URDF
+    es recomendable que los links tengan masa e inercia si más adelante se desea
+    llevar el modelo a simulación física.
+    Los valores son simplificados y no buscan una simulación dinámica realista.
   -->
   <xacro:macro name="simple_inertial" params="mass">
@@ -83,17 +198,29 @@
       <origin xyz="0 0 0" rpy="0 0 0"/>
       <mass value="${mass}"/>
-      <inertia ixx="0.001" ixy="0.0" ixz="0.0"
-               iyy="0.001" iyz="0.0"
-               izz="0.001"/>
+      <inertia
+        ixx="0.001" ixy="0.0" ixz="0.0"
+        iyy="0.001" iyz="0.0"
+        izz="0.001"/>
     </inertial>
   </xacro:macro>
-  <!-- ==================================================================== -->
-  <!-- 4. CUERPO PRINCIPAL (base_link)                                      -->
-  <!-- ==================================================================== -->
-  <!--
-    base_link es el marco de referencia central del dron.
-    Todos los demás elementos se anclan aquí.
-  -->
-  <link name="base_link">
+  <!-- ======================================================================= -->
+  <!-- 11. CUERPO CENTRAL DEL DRON                                             -->
+  <!-- ======================================================================= -->
+  <!--
+    base_link es el enlace principal del dron.
+    Todo el resto de piezas se conectan a base_link directa o indirectamente:
+      - brazos,
+      - motores,
+      - hélices,
+      - LED,
+      - patas.
+    Visual:
+      Dibuja una caja negra.
+    Collision:
+      Define una caja de colisión con la misma forma.
+    Inertial:
+      Añade una masa aproximada al cuerpo.
+  -->
+  <link name="${prefix}base_link">
     <visual>
       <geometry>
@@ -109,17 +236,39 @@
     <xacro:simple_inertial mass="1.2"/>
   </link>
-  <!-- ==================================================================== -->
-  <!-- 5. MACRO: MÓDULO BRAZO + MOTOR + HÉLICE (COMPLETO)                   -->
-  <!-- ==================================================================== -->
-  <!--
+  <!-- ======================================================================= -->
+  <!-- 12. MACRO PARA CREAR CADA BRAZO, MOTOR Y HÉLICE                         -->
+  <!-- ======================================================================= -->
+  <!--
+    Esta macro crea de una sola vez todo el conjunto de una esquina del dron:
+      1. Brazo diagonal.
+      2. Motor al final del brazo.
+      3. Buje central de la hélice.
+      4. Primera pala de la hélice.
+      5. Segunda pala de la hélice, girada 90 grados.
     Parámetros:
-      name: Identificador único (front_left, front_right, etc.)
-      x, y: Posición en el plano XY respecto a base_link
-      yaw: Rotación del brazo (para configuración X o +)
-      prop_material: Material a aplicar en las hélices (frontal/trasero)
+      name:
+        Nombre lógico de la esquina. Ejemplos:
+          front_left
+          front_right
+          rear_left
+          rear_right
+      x, y:
+        Posición del centro del brazo respecto a base_link.
+      yaw:
+        Giro del brazo alrededor del eje Z.
+        Esto permite colocar el brazo en diagonal.
+      prop_material:
+        Material/color de la hélice.
+        Las delanteras son rojas y las traseras azules.
   -->
   <xacro:macro name="arm_module" params="name x y yaw prop_material">
-    <!-- BRAZO -->
-    <link name="${name}_arm_link">
+    <!-- ==================================================================- -->
+    <!-- 12.1. Brazo diagonal                                                 -->
+    <!-- ==================================================================- -->
+    <!--
+      Dibuja una barra rectangular que sale del cuerpo hacia una esquina.
+      La barra está orientada mediante el yaw indicado en el joint.
+    -->
+    <link name="${prefix}${name}_arm_link">
       <visual>
         <geometry>
@@ -135,11 +284,20 @@
       <xacro:simple_inertial mass="0.10"/>
     </link>
-    <joint name="base_to_${name}_arm" type="fixed">
-      <parent link="base_link"/>
-      <child link="${name}_arm_link"/>
+    <!--
+      Une el brazo al cuerpo principal.
+      El giro yaw coloca el brazo en diagonal.
+    -->
+    <joint name="${prefix}base_to_${name}_arm" type="fixed">
+      <parent link="${prefix}base_link"/>
+      <child link="${prefix}${name}_arm_link"/>
       <origin xyz="${x} ${y} ${arm_z}" rpy="0 0 ${yaw}"/>
     </joint>
-    <!-- MOTOR -->
-    <link name="${name}_motor_link">
+    <!-- ==================================================================- -->
+    <!-- 12.2. Motor                                                          -->
+    <!-- ==================================================================- -->
+    <!--
+      Dibuja el motor como un cilindro vertical en el extremo exterior del brazo.
+    -->
+    <link name="${prefix}${name}_motor_link">
       <visual>
         <geometry>
@@ -155,11 +313,22 @@
       <xacro:simple_inertial mass="0.08"/>
     </link>
-    <joint name="${name}_arm_to_motor" type="fixed">
-      <parent link="${name}_arm_link"/>
-      <child link="${name}_motor_link"/>
+    <!--
+      Une el motor al extremo del brazo.
+      Como el motor depende del frame del brazo, su posición local se indica
+      respecto al centro del brazo.
+    -->
+    <joint name="${prefix}${name}_arm_to_motor" type="fixed">
+      <parent link="${prefix}${name}_arm_link"/>
+      <child link="${prefix}${name}_motor_link"/>
       <origin xyz="${arm_l/2.0 - motor_r/2.0} 0 ${arm_h/2.0 + motor_h/2.0}" rpy="0 0 0"/>
     </joint>
-    <!-- CUBO DE LA HÉLICE (HUB) -->
-    <link name="${name}_hub_link">
+    <!-- ==================================================================- -->
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